File: Humidity/PCB_project/Humidity_LED_Panel.kicad_pcb (KiCad board)
At the start: 2 copper layers, 238.8 x 135.9 mm, 1056 parts, among them J1 Signals, J2 PWR, U1 74HC595

Commit message: save new PWR
Parts:
- moved J1 10.0 mm to (134.0, 37.5) (x8)
- moved D2 10.0 mm to (221.6, 134.0) (x2)
- moved D2 10.0 mm to (97.2, 134.0) (x5)
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Other:
- board size 238.8 x 135.9 mm -> 248.3 x 139.1 mm
