File: Humidity/PCB_project/Humidity_Sensor_PWR.kicad_pcb (KiCad board)
At the start: 2 copper layers, 248.3 x 109.9 mm, 72 parts, among them J1 VCC_S, J2 VCC/GND, J3 GND_S

Commit message: save new PWR
Parts:
- removed the J1 at (95.9, 85.1)
- removed the J1 at (139.1, 113.7)
- removed the J1 at (53.3, 113.7)
- removed the J1 at (95.9, 113.7)
- removed the J1 at (95.9, 52.7)
- removed the J1 at (53.3, 52.7)
- removed the J1 at (139.1, 52.7)
- removed the J1 at (181.6, 52.7)
- removed the J1 at (266.1, 52.7)
- removed the J1 at (223.5, 52.7)
- removed the J1 at (223.5, 24.1)
- removed the J1 at (53.3, 85.1)
- removed the J1 at (266.1, 24.1)
- removed the J1 at (181.6, 24.1)
- removed the J1 at (139.1, 24.1)
- removed the J1 at (53.3, 24.1)
- removed the J1 at (95.9, 24.1)
- removed the J1 at (139.1, 85.1)
- removed the J1 at (181.6, 85.1)
- removed the J1 at (266.1, 85.1)
- removed the J1 at (223.5, 85.1)
- removed the J1 at (223.5, 113.7)
- removed the J1 at (266.1, 113.7)
- removed the J1 at (181.6, 113.7)
- removed the J2 at (80.0, 98.4)
- removed the J2 at (123.2, 127.0)
- removed the J2 at (37.5, 127.0)
- removed the J2 at (80.0, 127.0)
- removed the J2 at (80.0, 66.0)
- removed the J2 at (37.5, 66.0)
- removed the J2 at (123.2, 66.0)
- removed the J2 at (165.7, 66.0)
- removed the J2 at (250.2, 66.0)
- removed the J2 at (207.6, 66.0)
- removed the J2 at (207.6, 37.5)
- removed the J2 at (37.5, 98.4)
- removed the J2 at (250.2, 37.5)
- removed the J2 at (165.7, 37.5)
- removed the J2 at (123.2, 37.5)
- removed the J2 at (80.0, 37.5)
- removed the J2 at (123.2, 98.4)
- removed the J2 at (165.7, 98.4)
- removed the J2 at (250.2, 98.4)
- removed the J2 at (207.6, 98.4)
- removed the J2 at (207.6, 127.0)
- removed the J2 at (250.2, 127.0)
- removed the J2 at (165.7, 127.0)
- removed the J3 at (66.7, 85.1)
- removed the J3 at (109.9, 113.7)
- removed the J3 at (24.1, 113.7)
- removed the J3 at (66.7, 113.7)
- removed the J3 at (66.7, 52.7)
- removed the J3 at (24.1, 52.7)
- removed the J3 at (109.9, 52.7)
- removed the J3 at (152.4, 52.7)
- removed the J3 at (236.9, 52.7)
- removed the J3 at (194.3, 52.7)
- removed the J3 at (194.3, 24.1)
- removed the J3 at (24.1, 85.1)
- removed the J3 at (236.9, 24.1)
- removed the J3 at (152.4, 24.1)
- removed the J3 at (109.9, 24.1)
- removed the J3 at (24.1, 24.1)
- removed the J3 at (66.7, 24.1)
- removed the J3 at (109.9, 85.1)
- removed the J3 at (152.4, 85.1)
- removed the J3 at (236.9, 85.1)
- removed the J3 at (194.3, 85.1)
- removed the J3 at (194.3, 113.7)
- removed the J3 at (236.9, 113.7)
- removed the J3 at (152.4, 113.7)
- added J1 (x2): GND, Socket_Strips:Socket_Strip_Straight_1x05_Pitch2.54mm, F.Cu at (184.8, 33.7)
- added J1 (x2): GND, Socket_Strips:Socket_Strip_Straight_1x05_Pitch2.54mm, F.Cu at (235.6, 85.7)
- added J1 (x2): GND, Socket_Strips:Socket_Strip_Straight_1x05_Pitch2.54mm, F.Cu at (235.6, 110.5)
- added J1 (x2): GND, Socket_Strips:Socket_Strip_Straight_1x05_Pitch2.54mm, F.Cu at (235.6, 58.4)
- added J1 (x2): GND, Socket_Strips:Socket_Strip_Straight_1x05_Pitch2.54mm, F.Cu at (235.6, 33.7)
- added J1 (x2): GND, Socket_Strips:Socket_Strip_Straight_1x05_Pitch2.54mm, F.Cu at (123.2, 33.0)
- added J1 (x2): GND, Socket_Strips:Socket_Strip_Straight_1x05_Pitch2.54mm, F.Cu at (123.2, 57.8)
- added J1 (x2): GND, Socket_Strips:Socket_Strip_Straight_1x05_Pitch2.54mm, F.Cu at (123.2, 109.9)
- added J1 (x2): GND, Socket_Strips:Socket_Strip_Straight_1x05_Pitch2.54mm, F.Cu at (123.2, 85.1)
- added J1 (x2): GND, Socket_Strips:Socket_Strip_Straight_1x05_Pitch2.54mm, F.Cu at (72.4, 85.1)
- added J1 (x2): GND, Socket_Strips:Socket_Strip_Straight_1x05_Pitch2.54mm, F.Cu at (72.4, 109.9)
- added J1 (x2): GND, Socket_Strips:Socket_Strip_Straight_1x05_Pitch2.54mm, F.Cu at (72.4, 57.8)
- added J1 (x2): GND, Socket_Strips:Socket_Strip_Straight_1x05_Pitch2.54mm, F.Cu at (184.8, 58.4)
- added J1 (x2): GND, Socket_Strips:Socket_Strip_Straight_1x05_Pitch2.54mm, F.Cu at (72.4, 33.0)
- added J1 (x2): GND, Socket_Strips:Socket_Strip_Straight_1x05_Pitch2.54mm, F.Cu at (184.8, 110.5)
- added J1 (x2): GND, Socket_Strips:Socket_Strip_Straight_1x05_Pitch2.54mm, F.Cu at (184.8, 85.7)
- added J2 (x2): VCC/GND, Socket_Strips:Socket_Strip_Straight_1x02_Pitch2.54mm, F.Cu at (168.9, 47.0)
- added J2 (x2): VCC/GND, Socket_Strips:Socket_Strip_Straight_1x02_Pitch2.54mm, F.Cu at (219.7, 99.1)
- added J2 (x2): VCC/GND, Socket_Strips:Socket_Strip_Straight_1x02_Pitch2.54mm, F.Cu at (219.7, 123.8)
- added J2 (x2): VCC/GND, Socket_Strips:Socket_Strip_Straight_1x02_Pitch2.54mm, F.Cu at (219.7, 71.8)
- added J2 (x2): VCC/GND, Socket_Strips:Socket_Strip_Straight_1x02_Pitch2.54mm, F.Cu at (219.7, 47.0)
- added J2 (x2): VCC/GND, Socket_Strips:Socket_Strip_Straight_1x02_Pitch2.54mm, F.Cu at (107.3, 46.4)
- added J2 (x2): VCC/GND, Socket_Strips:Socket_Strip_Straight_1x02_Pitch2.54mm, F.Cu at (107.3, 71.1)
- added J2 (x2): VCC/GND, Socket_Strips:Socket_Strip_Straight_1x02_Pitch2.54mm, F.Cu at (107.3, 123.2)
- added J2 (x2): VCC/GND, Socket_Strips:Socket_Strip_Straight_1x02_Pitch2.54mm, F.Cu at (107.3, 98.4)
- added J2 (x2): VCC/GND, Socket_Strips:Socket_Strip_Straight_1x02_Pitch2.54mm, F.Cu at (56.5, 98.4)
- added J2 (x2): VCC/GND, Socket_Strips:Socket_Strip_Straight_1x02_Pitch2.54mm, F.Cu at (56.5, 123.2)
- added J2 (x2): VCC/GND, Socket_Strips:Socket_Strip_Straight_1x02_Pitch2.54mm, F.Cu at (56.5, 71.1)
- added J2 (x2): VCC/GND, Socket_Strips:Socket_Strip_Straight_1x02_Pitch2.54mm, F.Cu at (168.9, 71.8)
- added J2: VCC/GND, Socket_Strips:Socket_Strip_Straight_1x02_Pitch2.54mm, F.Cu at (56.5, 46.4)
- added J2 (x2): VCC/GND, Socket_Strips:Socket_Strip_Straight_1x02_Pitch2.54mm, F.Cu at (168.9, 123.8)
- added J2 (x2): VCC/GND, Socket_Strips:Socket_Strip_Straight_1x02_Pitch2.54mm, F.Cu at (168.9, 99.1)
- added J3 (x2): VCC, Socket_Strips:Socket_Strip_Straight_1x05_Pitch2.54mm, F.Cu at (155.6, 33.7)
- added J3 (x2): VCC, Socket_Strips:Socket_Strip_Straight_1x05_Pitch2.54mm, F.Cu at (206.4, 85.7)
- added J3 (x2): VCC, Socket_Strips:Socket_Strip_Straight_1x05_Pitch2.54mm, F.Cu at (206.4, 110.5)
- added J3 (x2): VCC, Socket_Strips:Socket_Strip_Straight_1x05_Pitch2.54mm, F.Cu at (206.4, 58.4)
- added J3 (x2): VCC, Socket_Strips:Socket_Strip_Straight_1x05_Pitch2.54mm, F.Cu at (206.4, 33.7)
- added J3 (x2): VCC, Socket_Strips:Socket_Strip_Straight_1x05_Pitch2.54mm, F.Cu at (94.0, 33.0)
- added J3 (x2): VCC, Socket_Strips:Socket_Strip_Straight_1x05_Pitch2.54mm, F.Cu at (94.0, 57.8)
- added J3 (x2): VCC, Socket_Strips:Socket_Strip_Straight_1x05_Pitch2.54mm, F.Cu at (94.0, 109.9)
- added J3 (x2): VCC, Socket_Strips:Socket_Strip_Straight_1x05_Pitch2.54mm, F.Cu at (94.0, 85.1)
- added J3 (x2): VCC, Socket_Strips:Socket_Strip_Straight_1x05_Pitch2.54mm, F.Cu at (43.2, 85.1)
- added J3 (x2): VCC, Socket_Strips:Socket_Strip_Straight_1x05_Pitch2.54mm, F.Cu at (43.2, 109.9)
- added J3 (x2): VCC, Socket_Strips:Socket_Strip_Straight_1x05_Pitch2.54mm, F.Cu at (43.2, 57.8)
- added J3 (x2): VCC, Socket_Strips:Socket_Strip_Straight_1x05_Pitch2.54mm, F.Cu at (155.6, 58.4)
- added J3 (x2): VCC, Socket_Strips:Socket_Strip_Straight_1x05_Pitch2.54mm, F.Cu at (43.2, 33.0)
- added J3 (x2): VCC, Socket_Strips:Socket_Strip_Straight_1x05_Pitch2.54mm, F.Cu at (155.6, 110.5)
- added J3 (x2): VCC, Socket_Strips:Socket_Strip_Straight_1x05_Pitch2.54mm, F.Cu at (155.6, 85.7)
- moved J2 21.0 mm to (56.5, 46.4)
Routing:
- net Net-(J1-Pad1): track 1630.2 -> 2645.9 mm
- net Net-(J2-Pad1): track 1676.0 -> 2686.6 mm
Other:
- board size 248.3 x 109.9 mm -> 198.8 x 97.8 mm
